Commit message: updates to simulation, attempting to add world files

File: simulation_ws/install/rover_sim/share/rover_sim/urdf/rover.urdf (robot description, URDF)
Before this commit: robot simple_rover, 5 links, 4 joints
Links:
- link base_link: mass 10.0 -> 5.0
Joints:
- joint wheel_fr_joint: axis 0 1 0 -> 0 -1 0
- joint wheel_rr_joint: axis 0 1 0 -> 0 -1 0
