Commit message: adding LiDAR plugin

File: simulation_ws/src/rover_sim/urdf/rover.urdf (robot description, URDF)
Before this commit: robot rover, 5 links, 4 joints
Links:
- added link lidar_link, mass 0.1; collision cylinder length=0.05 radius=0.05; visual cylinder length=0.05 radius=0.05
Joints:
- added joint lidar_joint: type fixed, parent base_link, child lidar_link, origin xyz=0 0 0.08 rpy=0 0 0

Commit message: scaled world and more tif cropping for different path lengths

File: simulation_ws/src/rover_sim/urdf/rover.urdf (robot description, URDF)
Before this commit: robot rover, 6 links, 5 joints
Joints:
- joint wheel_fl_joint: limit (none) -> effort=100 velocity=100
- joint wheel_fr_joint: limit (none) -> effort=100 velocity=100
- joint wheel_rl_joint: limit (none) -> effort=100 velocity=100
- joint wheel_rr_joint: limit (none) -> effort=100 velocity=100
